Commit message: Add jdcobot100 simulation workflow

File: onshape/jdcobot100/reference/jdcobot100.urdf (robot description, URDF)
Before this commit: robot jdcobot100_urdf, 5 links, 4 joints
Links:
- link arm_1_sub_asssembly: geometry collision mesh filename=package://assets/arm_1.stl; collision mesh filename=package://assets/sg90___micro_servo_9g___tower_pro_1_pe_a.s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
- link arm_2_sub_asssembly_copy_1: geometry collision mesh filename=package://assets/arm_1.stl; collision mesh filename=package://assets/sg90___micro_servo_9g___tower_pro_1_pe_a.s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
- link base_sub_assembly: geometry collision mesh filename=package://assets/base.stl; collision mesh filename=package://assets/base_link.stl
- link end_arm_sub_assembly: geometry collision mesh filename=package://assets/arm_end.stl; collision mesh filename=package://assets/sg90___micro_servo_9g___tower_pro_3_pe_a.s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
- link shoulder_sub_assembly: geometry collision mesh filename=package://assets/sg90___micro_servo_9g___tower_pro_1_pe_a.s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; collision mesh filename=package://assets/sg90___micro_servo_9g___tower_pro_1_pe_a__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
Joints:
- joint dof_base: limit lower=-0.523599 upper=0.523599 effort=10 velocity=1 -> lower=-3.141592653589793 upper=3.141592653589793 effort=10 velocity=10
- joint dof_elbow: limit lower=-0.523599 upper=0.523599 effort=10 velocity=1 -> lower=-3.141592653589793 upper=3.141592653589793 effort=10 velocity=10; origin xyz=-0.07515 -0 5.00002e-05 rpy=-0 0 0 -> xyz=-0.0506213 0.0555428 5.00002e-05 rpy=-0 -0 -0.831722
- joint dof_shoulder: limit lower=-0.523599 upper=0.523599 effort=10 velocity=1 -> lower=-3.141592653589793 upper=3.141592653589793 effort=10 velocity=10
- joint dof_wrist_pitch: limit lower=-0.523599 upper=0.523599 effort=10 velocity=1 -> lower=-3.141592653589793 upper=3.141592653589793 effort=10 velocity=10; origin xyz=-0.07515 -0 5.00002e-05 rpy=0 -0 0 -> xyz=0.00122811 -0.07514 5.00002e-05 rpy=0 0 1.58714

File: ros_arm/urdf/ros_arm_gazebo.urdf (robot description, URDF)
Before this commit: robot ros_arm_gazebo, 6 links, 5 joints
Joints:
- removed joint arm1_arm2
- removed joint arn2_end_arm
- removed joint base_shoulder
- removed joint shoulder_arm1
- added joint dof_base: type revolute, parent base_sub_assembly, child shoulder_sub_assembly, origin xyz=0 0 0.05, axis 0 0 1, limit lower=-0.523599 upper=0.523599 effort=2.0 velocity=1.0
- added joint dof_elbow: type revolute, parent arm_1_sub_asssembly, child arm_2_sub_asssembly_copy_1, origin xyz=0.12 0 0, axis 0 1 0, limit lower=-0.523599 upper=0.523599 effort=1.5 velocity=1.0
- added joint dof_shoulder: type revolute, parent shoulder_sub_assembly, child arm_1_sub_asssembly, origin xyz=0 0 0.07, axis 0 1 0, limit lower=-0.523599 upper=0.523599 effort=2.0 velocity=1.0
- added joint dof_wrist_pitch: type revolute, parent arm_2_sub_asssembly_copy_1, child end_arm_sub_assembly, origin xyz=0.11 0 0, axis 0 1 0, limit lower=-0.523599 upper=0.523599 effort=1.0 velocity=1.0
